File: electrical/ElectricalSchematic/ElectricalSchematic.sch (KiCad schematic (older format))
At the start: 12 parts

Commit message: electrical updates
Parts:
- removed M?: Motor_Servo, symbol Motor:Motor_Servo
Connections:
- net labels removed: Servo2
- wire segments 89 -> 79
Other:
- note removed: "Drives the balance control"
Changed lines of the file:
@@
 EESchema Schematic File Version 4
+LIBS:ElectricalSchematic-cache
 EELAYER 30 0
 EELAYER END
@@
 Wire Wire Line
 	8900 1900 8900 1650
-Connection ~ 8900 1900
 Wire Wire Line
 	9100 1900 8900 1900
 Wire Wire Line
-	8900 2450 8900 1900
-Wire Wire Line
-	9100 2450 8900 2450
-Wire Wire Line
-	8800 2000 8800 2550
-Wire Wire Line
-	8800 2550 8800 2750
-Connection ~ 8800 2550
-Wire Wire Line
-	9100 2550 8800 2550
-Wire Wire Line
-	9100 2000 8800 2000
-$Comp
-L power:GND #PWR?
-U 1 1 5DC957BD
-P 8800 2750
-F 0 "#PWR?" H 8800 2500 50  0001 C CNN
-F 1 "GND" H 8805 2577 50  0000 C CNN
-F 2 "" H 8800 2750 50  0001 C CNN
-F 3 "" H 8800 2750 50  0001 C CNN
-	1    8800 2750
-	1    0    0    -1
-$EndComp
-Text Notes 9250 2200 0    50   ~ 0
-Drives the balance control
-$Comp
-L Motor:Motor_Servo M?
-U 1 1 5DC8DF14
-P 9400 2450
-F 0 "M?" H 9732 2515 50  0000 L CNN
-F 1 "Motor_Servo" H 9732 2424 50  0000 L CNN
-F 2 "" H 9400 2260 50  0001 C CNN
-F 3 "http://forums.parallax.com/uploads/attachments/46831/74481.png" H 9400 2260 50  0001 C CNN
-	1    9400 2450
-	1    0    0    -1
-$EndComp
+	9100 2000 8900 2000
 $Comp
 L Motor:Motor_Servo M?
@@
 $EndComp
 Wire Wire Line
+	7050 1700 7050 1500
+Wire Wire Line
+	7050 1800 7050 1900
+Wire Wire Line
+	8550 1800 9100 1800
+Wire Wire Line
+	5150 3000 5150 4950
+Wire Wire Line
+	5150 4950 4700 4950
+Wire Wire Line
+	4700 5050 7100 5050
+Wire Wire Line
+	7100 5050 7100 4250
+Wire Wire Line
+	7100 4250 7750 4250
+Wire Wire Line
+	7750 4350 7200 4350
+Wire Wire Line
+	7200 4350 7200 5150
+Wire Wire Line
+	7200 5150 4700 5150
+Wire Wire Line
+	4700 5250 7150 5250
+Wire Wire Line
+	7150 5250 7150 5600
+Wire Wire Line
+	7150 5600 7750 5600
+Wire Wire Line
+	7750 5700 7050 5700
+Wire Wire Line
+	7050 5700 7050 5350
+Wire Wire Line
+	7050 5350 4700 5350
+Wire Wire Line
+	4700 5650 5100 5650
+Text Label 4800 5650 0    50   ~ 0
+Servo1
+$Comp
+L 11.1V:GND #PWR?
+U 1 1 5DD84ACB
+P 8900 2150
+F 0 "#PWR?" H 8900 1900 50  0001 C CNN
+F 1 "GND" H 8905 1977 50  0000 C CNN
+F 2 "" H 8900 2150 50  0001 C CNN
+F 3 "" H 8900 2150 50  0001 C CNN
+	1    8900 2150
+	1    0    0    -1
+$EndComp
+Wire Wire Line
+	8900 2000 8900 2150
+Wire Wire Line
+	7250 1800 7050 1800
+Wire Wire Line
 	7250 1700 7050 1700
 Wire Wire Line
-	7050 1700 7050 1500
+	8250 1900 8250 2250
+Text Label 8250 2200 1    50   ~ 0
+Servo1
+Wire Wire Line
+	8250 2250 8550 2250
+Wire Wire Line
+	8100 2250 8250 2250
 $Comp
 L 11.1V:MotorShield_simplified U?
@@
 	1    0    0    -1
 $EndComp
-Wire Wire Line
-	7250 1800 7050 1800
-Wire Wire Line
-	7050 1800 7050 1900
-Wire Wire Line
-	8100 2150 8250 2150
-Wire Wire Line
-	8550 2150 8550 1800
-Wire Wire Line
-	8550 1800 9100 1800
-Wire Wire Line
-	8550 2250 8550 2350
-Wire Wire Line
-	8550 2350 9100 2350
-Wire Wire Line
-	5150 3000 5150 4950
-Wire Wire Line
-	5150 4950 4700 4950
-Wire Wire Line
-	4700 5050 7100 5050
-Wire Wire Line
-	7100 5050 7100 4250
-Wire Wire Line
-	7100 4250 7750 4250
-Wire Wire Line
-	7750 4350 7200 4350
-Wire Wire Line
-	7200 4350 7200 5150
-Wire Wire Line
-	7200 5150 4700 5150
-Wire Wire Line
-	4700 5250 7150 5250
-Wire Wire Line
-	7150 5250 7150 5600
-Wire Wire Line
-	7150 5600 7750 5600
-Wire Wire Line
-	7750 5700 7050 5700
-Wire Wire Line
-	7050 5700 7050 5350
-Wire Wire Line
-	7050 5350 4700 5350
-Connection ~ 8250 2150
-Wire Wire Line
-	8250 2150 8550 2150
-Wire Wire Line
-	8100 2250 8250 2250
-Text Label 8250 2100 1    50   ~ 0
-Servo1
-Text Label 8250 2550 1    50   ~ 0
-Servo2
-Wire Wire Line
-	8250 1800 8250 2150
-Wire Wire Line
-	8250 2250 8250 2650
 Connection ~ 8250 2250
 Wire Wire Line
-	8250 2250 8550 2250
-Wire Wire Line
-	4700 5650 5100 5650
-Wire Wire Line
-	4700 5750 5100 5750
+	8550 1800 8550 2250
 Wire Bus Line
 	3250 3900 4650 3900
-Text Label 4800 5750 0    50   ~ 0
-Servo2
-Text Label 4800 5650 0    50   ~ 0
-Servo1
 $EndSCHEMATC

Commit message: electrical updates
Parts:
- added F? (x2): Fuse, symbol Device:Fuse
Changed lines of the file:
@@
 Wire Wire Line
 	9050 3850 9450 3850
-Wire Wire Line
-	8450 4450 8650 4450
-Wire Wire Line
-	8650 4450 8650 3750
-Wire Wire Line
-	8650 4450 8650 5800
-Wire Wire Line
-	8650 5800 8450 5800
-Connection ~ 8650 4450
 $Comp
 L 11.1V:+11.1V #PWR?
 U 1 1 5DC86ADF
-P 8650 3750
-F 0 "#PWR?" H 8650 3600 50  0001 C CNN
-F 1 "+11.1V" H 8665 3923 50  0000 C CNN
-F 2 "" H 8650 3750 50  0001 C CNN
-F 3 "" H 8650 3750 50  0001 C CNN
-	1    8650 3750
+P 8850 3750
+F 0 "#PWR?" H 8850 3600 50  0001 C CNN
+F 1 "+11.1V" H 8865 3923 50  0000 C CNN
+F 2 "" H 8850 3750 50  0001 C CNN
+F 3 "" H 8850 3750 50  0001 C CNN
+	1    8850 3750
 	1    0    0    -1
 $EndComp
@@
 Wire Wire Line
 	8550 1800 8550 2250
+Wire Wire Line
+	8850 3750 8850 4450
+$Comp
+L Device:Fuse F?
+U 1 1 5DDA0F62
+P 8700 4450
+F 0 "F?" V 8503 4450 50  0000 C CNN
+F 1 "Fuse" V 8594 4450 50  0000 C CNN
+F 2 "" V 8630 4450 50  0001 C CNN
+F 3 "~" H 8700 4450 50  0001 C CNN
+	1    8700 4450
+	0    1    1    0
+$EndComp
+$Comp
+L Device:Fuse F?
+U 1 1 5DDA2E37
+P 8700 5800
+F 0 "F?" V 8503 5800 50  0000 C CNN
+F 1 "Fuse" V 8594 5800 50  0000 C CNN
+F 2 "" V 8630 5800 50  0001 C CNN
+F 3 "~" H 8700 5800 50  0001 C CNN
+	1    8700 5800
+	0    1    1    0
+$EndComp
+Connection ~ 8850 4450
+Wire Wire Line
+	8850 4450 8850 5800
+Wire Wire Line
+	8550 4450 8450 4450
+Wire Wire Line
+	8550 5800 8450 5800
 Wire Bus Line
 	3250 3900 4650 3900
